File: untitled.kicad_sch (KiCad schematic)
At the start: 0 parts

Commit message: version update
Parts:
- added D2: LED, symbol Device:LED
- added J3: Conn_01x02_Socket, symbol Connector:Conn_01x02_Socket
- added R1: R_US, symbol Device:R_US
- added SW2: SW_Push, symbol Switch:SW_Push
Connections:
- new net: R1.1, SW2.1
- new net +5V: SW2.2
- new net GND: D2.1 (K), J3.2 (Pin_2)
- new net V_led: D2.2 (A), J3.1 (Pin_1), R1.2
Changed lines of the file:
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@@
 (kicad_sch (version 20230121) (generator eeschema)
   (paper "A4")
+  (junction (at 196.85 113.03) (diameter 0) (color 0 0 0 0)
+  )
+  (junction (at 198.12 127) (diameter 0) (color 0 0 0 0)
+  )
+  (wire (pts (xy 123.19 113.03) (xy 196.85 113.03))
+    (stroke (width 0) (type default))
+  )
+  (wire (pts (xy 196.85 124.46) (xy 196.85 113.03))
+    (stroke (width 0) (type default))
+  )
+  (wire (pts (xy 123.19 62.23) (xy 123.19 76.2))
+    (stroke (width 0) (type default))
+  )
+  (wire (pts (xy 207.01 113.03) (xy 207.01 116.84))
+    (stroke (width 0) (type default))
+  )
+  (wire (pts (xy 123.19 86.36) (xy 123.19 105.41))
+    (stroke (width 0) (type default))
+  )
+  (wire (pts (xy 198.12 127) (xy 196.85 127))
+    (stroke (width 0) (type default))
+  )
+  (wire (pts (xy 196.85 113.03) (xy 207.01 113.03))
+    (stroke (width 0) (type default))
+  )
+  (wire (pts (xy 207.01 124.46) (xy 207.01 127))
+    (stroke (width 0) (type default))
+  )
+  (wire (pts (xy 207.01 127) (xy 198.12 127))
+    (stroke (width 0) (type default))
+  )
+  (hierarchical_label "V_led" (shape input) (at 196.85 113.03 90) (fields_autoplaced)
+    (effects (font (size 1.27 1.27)) (justify left))
+  )
+  (symbol (lib_id "power:GND") (at 198.12 127 0) (unit 1)
+    (in_bom yes) (on_board yes) (dnp no) (fields_autoplaced)
+    (property "Reference" "#PWR07" (at 198.12 133.35 0)
+      (effects (font (size 1.27 1.27)) hide)
+    )
+    (property "Value" "GND" (at 198.12 132.08 0)
+      (effects (font (size 1.27 1.27)))
+    )
+    (property "Footprint" "" (at 198.12 127 0)
+      (effects (font (size 1.27 1.27)) hide)
+    )
+    (property "Datasheet" "" (at 198.12 127 0)
+      (effects (font (size 1.27 1.27)) hide)
+    )
+    (pin "1")
+    (instances
+      (project "voltage_regulated_led_new"
+        (path "/7d837360-0bad-4c76-8645-e18e924dfa75/fdc9af70-ef5e-43c1-851d-2201b5fa75d7"
+          (reference "#PWR07") (unit 1)
+        )
+      )
+    )
+  )
+  (symbol (lib_id "Connector:Conn_01x02_Socket") (at 191.77 124.46 0) (mirror y) (unit 1)
+    (in_bom yes) (on_board yes) (dnp no)
+    (property "Reference" "J3" (at 190.5 124.46 0)
+      (effects (font (size 1.27 1.27)) (justify left))
+    )
+    (property "Value" "Conn_01x02_Socket" (at 190.5 127 0)
+      (effects (font (size 1.27 1.27)) (justify left))
+    )
+    (property "Footprint" "" (at 191.77 124.46 0)
+      (effects (font (size 1.27 1.27)) hide)
+    )
+    (property "Datasheet" "~" (at 191.77 124.46 0)
+      (effects (font (size 1.27 1.27)) hide)
+    )
+    (pin "1")
+    (pin "2")
+    (instances
+      (project "voltage_regulated_led_new"
+        (path "/7d837360-0bad-4c76-8645-e18e924dfa75/fdc9af70-ef5e-43c1-851d-2201b5fa75d7"
+          (reference "J3") (unit 1)
+        )
+      )
+    )
+  )
+  (symbol (lib_id "power:+5V") (at 123.19 62.23 0) (unit 1)
+    (in_bom yes) (on_board yes) (dnp no) (fields_autoplaced)
+    (property "Reference" "#PWR06" (at 123.19 66.04 0)
+      (effects (font (size 1.27 1.27)) hide)
+    )
+    (property "Value" "+5V" (at 123.19 57.15 0)
+      (effects (font (size 1.27 1.27)))
+    )
+    (property "Footprint" "" (at 123.19 62.23 0)
+      (effects (font (size 1.27 1.27)) hide)
+    )
+    (property "Datasheet" "" (at 123.19 62.23 0)
+      (effects (font (size 1.27 1.27)) hide)
+    )
+    (pin "1")
+    (instances
+      (project "voltage_regulated_led_new"
+        (path "/7d837360-0bad-4c76-8645-e18e924dfa75/fdc9af70-ef5e-43c1-851d-2201b5fa75d7"
+          (reference "#PWR06") (unit 1)
+        )
+      )
+    )
+  )
+  (symbol (lib_id "Device:LED") (at 207.01 120.65 90) (unit 1)
+    (in_bom yes) (on_board yes) (dnp no) (fields_autoplaced)
+    (property "Reference" "D2" (at 210.82 120.9675 90)
+      (effects (font (size 1.27 1.27)) (justify right))
+    )
+    (property "Value" "LED" (at 210.82 123.5075 90)
+      (effects (font (size 1.27 1.27)) (justify right))
+    )
+    (property "Footprint" "" (at 207.01 120.65 0)
+      (effects (font (size 1.27 1.27)) hide)
+    )
+    (property "Datasheet" "~" (at 207.01 120.65 0)
+      (effects (font (size 1.27 1.27)) hide)
+    )
+    (pin "1")
+    (pin "2")
+    (instances
+      (project "voltage_regulated_led_new"
+        (path "/7d837360-0bad-4c76-8645-e18e924dfa75/fdc9af70-ef5e-43c1-851d-2201b5fa75d7"
+          (reference "D2") (unit 1)
+        )
+      )
+    )
+  )
+  (symbol (lib_id "Switch:SW_Push") (at 123.19 81.28 90) (unit 1)
+    (in_bom yes) (on_board yes) (dnp no) (fields_autoplaced)
+    (property "Reference" "SW2" (at 124.46 80.01 90)
+      (effects (font (size 1.27 1.27)) (justify right))
+    )
+    (property "Value" "SW_Push" (at 124.46 82.55 90)
+      (effects (font (size 1.27 1.27)) (justify right))
+    )
+    (property "Footprint" "" (at 118.11 81.28 0)
+      (effects (font (size 1.27 1.27)) hide)
+    )
+    (property "Datasheet" "~" (at 118.11 81.28 0)
+      (effects (font (size 1.27 1.27)) hide)
+    )
+    (pin "1")
+    (pin "2")
+    (instances
+      (project "voltage_regulated_led_new"
+        (path "/7d837360-0bad-4c76-8645-e18e924dfa75/fdc9af70-ef5e-43c1-851d-2201b5fa75d7"
+          (reference "SW2") (unit 1)
+        )
+      )
+    )
+  )
+  (symbol (lib_id "Device:R_US") (at 123.19 109.22 0) (unit 1)
+    (in_bom yes) (on_board yes) (dnp no) (fields_autoplaced)
+    (property "Reference" "R1" (at 125.73 107.95 0)
+      (effects (font (size 1.27 1.27)) (justify left))
+    )
+    (property "Value" "R_US" (at 125.73 110.49 0)
+      (effects (font (size 1.27 1.27)) (justify left))
+    )
+    (property "Footprint" "" (at 124.206 109.474 90)
+      (effects (font (size 1.27 1.27)) hide)
+    )
+    (property "Datasheet" "~" (at 123.19 109.22 0)
+      (effects (font (size 1.27 1.27)) hide)
+    )
+    (pin "1")
+    (pin "2")
+    (instances
+      (project "voltage_regulated_led_new"
+        (path "/7d837360-0bad-4c76-8645-e18e924dfa75/fdc9af70-ef5e-43c1-851d-2201b5fa75d7"
+          (reference "R1") (unit 1)
+        )
+      )
+    )
+  )
 )
