File: voltage_regulated_led_new.kicad_sch (KiCad schematic)
At the start: 13 parts, among them J1 Conn_01x02_Socket, J2 Conn_01x06_Pin, J4 Conn_01x02_Socket, SW1 SW_SPST, U1 LM7805_TO220

Commit message: version update
Parts:
- removed H1, H2, H3, H4: MountingHole, MountingHole:MountingHole_2.2mm_M2, symbol Mechanical:MountingHole
- removed J2: Conn_01x06_Pin, Connector_PinSocket_2.54mm:PinSocket_1x06_P2.54mm_Vertical, symbol Connector:Conn_01x06_Pin
- removed J4: Conn_01x02_Socket, symbol Connector:Conn_01x02_Socket
- added J2: Conn_01x04_Pin, symbol Connector:Conn_01x04_Pin
- C1, C2: footprint Capacitor_THT:CP_Axial_L10.0mm_D4.5mm_P15.00mm_Horizontal -> (none)
- D1: footprint LED_THT:LED_D3.0mm_Horizontal_O1.27mm_Z10.0mm -> (none)
- J1: footprint Connector_PinHeader_2.54mm:PinHeader_1x02_P2.54mm_Vertical -> (none)
- SW1: footprint Button_Switch_THT:SW_DIP_SPSTx01_Piano_10.8x4.1mm_W7.62mm_P2.54mm -> (none)
Connections:
- net +9V: now also SW1.1 (A)
- net +9v: now also J2.4 (Pin_4); no longer SW1.2 (B)
- net GND: now also J2.2 (Pin_2), J2.3 (Pin_3); no longer D1.2 (A), SW1.1 (A)
- new net: D1.2 (A), SW1.2 (B)
- new net V_led: J2.1 (Pin_1)
Other:
- sheet Push-Button Activated LED ports: added none; removed Vled
- moved on the sheet: SW1

Commit message: update
Parts:
- C1, C2: footprint (none) -> Capacitor_THT:CP_Axial_L10.0mm_D4.5mm_P15.00mm_Horizontal
- D1: footprint (none) -> LED_THT:LED_D3.0mm_Horizontal_O1.27mm_Z10.0mm
- SW1: footprint (none) -> Button_Switch_THT:SW_DIP_SPSTx01_Piano_10.8x4.1mm_W7.62mm_P2.54mm
Connections:
- net V_led renamed Push-Button Activated LED/Vled
Other:
- sheet Push-Button Activated LED ports: added Vled; removed none
Changed lines of the file:
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@@
     (stroke (width 0) (type default))
   )
-  (wire (pts (xy 133.35 135.89) (xy 194.31 135.89))
+  (wire (pts (xy 133.35 135.89) (xy 187.96 135.89))
     (stroke (width 0) (type default))
   )
@@
   )
   (wire (pts (xy 127 71.12) (xy 127 64.77))
-    (stroke (width 0) (type default))
-  )
-  (wire (pts (xy 194.31 135.89) (xy 194.31 140.97))
     (stroke (width 0) (type default))
   )
@@
     (effects (font (size 1.27 1.27)) (justify left bottom))
   )
-  (hierarchical_label "V_led" (shape input) (at 194.31 140.97 0) (fields_autoplaced)
-    (effects (font (size 1.27 1.27)) (justify left))
-  )
   (symbol (lib_id "power:+9V") (at 80.01 64.77 0) (unit 1)
     (in_bom yes) (on_board yes) (dnp no) (fields_autoplaced)
@@
   )
   (symbol (lib_id "Connector:Conn_01x02_Socket") (at 63.5 77.47 0) (unit 1)
-    (in_bom yes) (on_board yes) (dnp no) (fields_autoplaced)
+    (in_bom yes) (on_board no) (dnp no) (fields_autoplaced)
     (property "Reference" "J1" (at 64.77 77.47 0)
       (effects (font (size 1.27 1.27)) (justify left))
@@
       (effects (font (size 1.27 1.27)) (justify left))
     )
-    (property "Footprint" "" (at 181.61 78.74 0)
+    (property "Footprint" "Capacitor_THT:CP_Axial_L10.0mm_D4.5mm_P15.00mm_Horizontal" (at 181.61 78.74 0)
       (effects (font (size 1.27 1.27)) hide)
     )
@@
       (effects (font (size 1.27 1.27)))
     )
-    (property "Footprint" "" (at 113.03 64.77 0)
+    (property "Footprint" "LED_THT:LED_D3.0mm_Horizontal_O1.27mm_Z10.0mm" (at 113.03 64.77 0)
       (effects (font (size 1.27 1.27)) hide)
     )
@@
   )
   (symbol (lib_id "power:GND") (at 58.42 83.82 0) (unit 1)
-    (in_bom yes) (on_board yes) (dnp no) (fields_autoplaced)
+    (in_bom yes) (on_board no) (dnp no) (fields_autoplaced)
     (property "Reference" "#PWR04" (at 58.42 90.17 0)
       (effects (font (size 1.27 1.27)) hide)
@@
       (effects (font (size 1.27 1.27)) (justify left))
     )
-    (property "Footprint" "" (at 127 80.01 0)
+    (property "Footprint" "Capacitor_THT:CP_Axial_L10.0mm_D4.5mm_P15.00mm_Horizontal" (at 127 80.01 0)
       (effects (font (size 1.27 1.27)) hide)
     )
@@
   )
   (symbol (lib_id "Connector:Conn_01x04_Pin") (at 130.81 143.51 270) (mirror x) (unit 1)
-    (in_bom yes) (on_board yes) (dnp no) (fields_autoplaced)
+    (in_bom yes) (on_board no) (dnp no) (fields_autoplaced)
     (property "Reference" "J2" (at 129.54 148.59 90)
       (effects (font (size 1.27 1.27)))
@@
       (effects (font (size 1.27 1.27)))
     )
-    (property "Footprint" "" (at 95.25 64.77 0)
+    (property "Footprint" "Button_Switch_THT:SW_DIP_SPSTx01_Piano_10.8x4.1mm_W7.62mm_P2.54mm" (at 95.25 64.77 0)
       (effects (font (size 1.27 1.27)) hide)
     )
@@
   )
   (symbol (lib_id "power:GND") (at 129.54 133.35 0) (mirror x) (unit 1)
-    (in_bom yes) (on_board yes) (dnp no) (fields_autoplaced)
+    (in_bom yes) (on_board no) (dnp no) (fields_autoplaced)
     (property "Reference" "#PWR05" (at 129.54 127 0)
       (effects (font (size 1.27 1.27)) hide)
@@
   )
   (symbol (lib_id "Device:Battery") (at 43.18 78.74 0) (unit 1)
-    (in_bom yes) (on_board yes) (dnp no) (fields_autoplaced)
+    (in_bom yes) (on_board no) (dnp no) (fields_autoplaced)
     (property "Reference" "BT1" (at 46.99 76.8985 0)
       (effects (font (size 1.27 1.27)) (justify left))
@@
     )
   )
-  (sheet (at 184.15 115.57) (size 43.18 35.56) (fields_autoplaced)
+  (sheet (at 187.96 111.76) (size 35.56 43.18) (fields_autoplaced)
     (stroke (width 0.1524) (type solid))
     (fill (color 0 0 0 0.0000))
-    (property "Sheetname" "Push-Button Activated LED" (at 184.15 114.8584 0)
+    (property "Sheetname" "Push-Button Activated LED" (at 187.2484 154.94 90)
       (effects (font (size 1.27 1.27)) (justify left bottom))
     )
-    (property "Sheetfile" "untitled.kicad_sch" (at 184.15 151.7146 0)
+    (property "Sheetfile" "untitled.kicad_sch" (at 224.1046 154.94 90)
       (effects (font (size 1.27 1.27)) (justify left top))
     )
-    (instances
+    (pin "Vled" input (at 187.96 135.89 180)
+      (effects (font (size 1.27 1.27)) (justify left))
+    )
+    (instances
