File: NEW NEW/untitled.kicad_sch (KiCad schematic)
At the start: 4 parts, among them J3 Conn_01x02_Socket, SW2 SW_Push

Commit message: real edits this time!
Parts:
- added J5: Conn_01x02_Socket, symbol Connector:Conn_01x02_Socket
Connections:
- net +5V: now also J5.2 (Pin_2)
- net GND: now also R1.1, SW2.1, J5.1 (Pin_1)
Other:
- moved on the sheet: SW2
Changed lines of the file:
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@@
   (junction (at 196.85 113.03) (diameter 0) (color 0 0 0 0)
   )
+  (junction (at 95.25 74.93) (diameter 0) (color 0 0 0 0)
+  )
   (junction (at 198.12 127) (diameter 0) (color 0 0 0 0)
   )
+  (junction (at 95.25 88.9) (diameter 0) (color 0 0 0 0)
+  )
   (wire (pts (xy 123.19 113.03) (xy 196.85 113.03))
     (stroke (width 0) (type default))
@@
     (stroke (width 0) (type default))
   )
-  (wire (pts (xy 123.19 62.23) (xy 123.19 76.2))
-    (stroke (width 0) (type default))
-  )
   (wire (pts (xy 207.01 113.03) (xy 207.01 116.84))
     (stroke (width 0) (type default))
   )
-  (wire (pts (xy 123.19 86.36) (xy 123.19 105.41))
+  (wire (pts (xy 104.14 88.9) (xy 104.14 85.09))
+    (stroke (width 0) (type default))
+  )
+  (wire (pts (xy 95.25 81.28) (xy 95.25 88.9))
+    (stroke (width 0) (type default))
+  )
+  (wire (pts (xy 123.19 74.93) (xy 123.19 62.23))
     (stroke (width 0) (type default))
   )
@@
     (stroke (width 0) (type default))
   )
+  (wire (pts (xy 95.25 74.93) (xy 104.14 74.93))
+    (stroke (width 0) (type default))
+  )
   (wire (pts (xy 196.85 113.03) (xy 207.01 113.03))
     (stroke (width 0) (type default))
@@
     (stroke (width 0) (type default))
   )
+  (wire (pts (xy 123.19 88.9) (xy 123.19 105.41))
+    (stroke (width 0) (type default))
+  )
+  (wire (pts (xy 95.25 88.9) (xy 104.14 88.9))
+    (stroke (width 0) (type default))
+  )
   (wire (pts (xy 207.01 127) (xy 198.12 127))
+    (stroke (width 0) (type default))
+  )
+  (wire (pts (xy 95.25 78.74) (xy 95.25 74.93))
     (stroke (width 0) (type default))
   )
@@
     )
   )
+  (symbol (lib_id "Connector:Conn_01x02_Socket") (at 90.17 81.28 180) (unit 1)
+    (in_bom yes) (on_board yes) (dnp no) (fields_autoplaced)
+    (property "Reference" "J5" (at 90.805 73.66 0)
+      (effects (font (size 1.27 1.27)))
+    )
+    (property "Value" "Conn_01x02_Socket" (at 90.805 76.2 0)
+      (effects (font (size 1.27 1.27)))
+    )
+    (property "Footprint" "" (at 90.17 81.28 0)
+      (effects (font (size 1.27 1.27)) hide)
+    )
+    (property "Datasheet" "~" (at 90.17 81.28 0)
+      (effects (font (size 1.27 1.27)) hide)
+    )
+    (pin "1")
+    (pin "2")
+    (instances
+      (project "voltage_regulated_led_new"
+        (path "/7d837360-0bad-4c76-8645-e18e924dfa75/fdc9af70-ef5e-43c1-851d-2201b5fa75d7"
+          (reference "J5") (unit 1)
+        )
+      )
+    )
+  )
   (symbol (lib_id "Connector:Conn_01x02_Socket") (at 191.77 124.46 0) (mirror y) (unit 1)
     (in_bom yes) (on_board no) (dnp no)
@@
     )
   )
+  (symbol (lib_id "power:GND") (at 123.19 88.9 90) (unit 1)
+    (in_bom yes) (on_board yes) (dnp no) (fields_autoplaced)
+    (property "Reference" "#PWR010" (at 129.54 88.9 0)
+      (effects (font (size 1.27 1.27)) hide)
+    )
+    (property "Value" "GND" (at 127 88.9 90)
+      (effects (font (size 1.27 1.27)) (justify right))
+    )
+    (property "Footprint" "" (at 123.19 88.9 0)
+      (effects (font (size 1.27 1.27)) hide)
+    )
+    (property "Datasheet" "" (at 123.19 88.9 0)
+      (effects (font (size 1.27 1.27)) hide)
+    )
+    (pin "1")
+    (instances
+      (project "voltage_regulated_led_new"
+        (path "/7d837360-0bad-4c76-8645-e18e924dfa75/fdc9af70-ef5e-43c1-851d-2201b5fa75d7"
+          (reference "#PWR010") (unit 1)
+        )
+      )
+    )
+  )
+  (symbol (lib_id "power:+5V") (at 95.25 74.93 0) (unit 1)
+    (in_bom yes) (on_board yes) (dnp no) (fields_autoplaced)
+    (property "Reference" "#PWR012" (at 95.25 78.74 0)
+      (effects (font (size 1.27 1.27)) hide)
+    )
+    (property "Value" "+5V" (at 95.25 69.85 0)
+      (effects (font (size 1.27 1.27)))
+    )
+    (property "Footprint" "" (at 95.25 74.93 0)
+      (effects (font (size 1.27 1.27)) hide)
+    )
+    (property "Datasheet" "" (at 95.25 74.93 0)
+      (effects (font (size 1.27 1.27)) hide)
+    )
+    (pin "1")
+    (instances
+      (project "voltage_regulated_led_new"
+        (path "/7d837360-0bad-4c76-8645-e18e924dfa75/fdc9af70-ef5e-43c1-851d-2201b5fa75d7"
+          (reference "#PWR012") (unit 1)
+        )
+      )
+    )
+  )
   (symbol (lib_id "Device:LED") (at 207.01 120.65 90) (unit 1)
     (in_bom yes) (on_board no) (dnp no) (fields_autoplaced)
@@
     )
   )
-  (symbol (lib_id "Switch:SW_Push") (at 123.19 81.28 90) (unit 1)
-    (in_bom yes) (on_board yes) (dnp no) (fields_autoplaced)
-    (property "Reference" "SW2" (at 124.46 80.01 90)
-      (effects (font (size 1.27 1.27)) (justify right))
-    )
-    (property "Value" "SW_Push" (at 124.46 82.55 90)
-      (effects (font (size 1.27 1.27)) (justify right))
-    )
-    (property "Footprint" "Button_Switch_THT:Push_E-Switch_KS01Q01" (at 118.11 81.28 0)
-      (effects (font (size 1.27 1.27)) hide)
-    )
-    (property "Datasheet" "~" (at 118.11 81.28 0)
+  (symbol (lib_id "Switch:SW_Push") (at 104.14 80.01 90) (unit 1)
+    (in_bom yes) (on_board yes) (dnp no) (fields_autoplaced)
+    (property "Reference" "SW2" (at 105.41 78.74 90)
+      (effects (font (size 1.27 1.27)) (justify right))
+    )
+    (property "Value" "SW_Push" (at 105.41 81.28 90)
+      (effects (font (size 1.27 1.27)) (justify right))
+    )
+    (property "Footprint" "Button_Switch_THT:Push_E-Switch_KS01Q01" (at 99.06 80.01 0)
+      (effects (font (size 1.27 1.27)) hide)
+    )
+    (property "Datasheet" "~" (at 99.06 80.01 0)
       (effects (font (size 1.27 1.27)) hide)
     )
@@
         )
       )
+    )
+  )
+  (symbol (lib_id "power:GND") (at 95.25 88.9 0) (unit 1)
+    (in_bom yes) (on_board yes) (dnp no) (fields_autoplaced)
+    (property "Reference" "#PWR011" (at 95.25 95.25 0)
+      (effects (font (size 1.27 1.27)) hide)
+    )
+    (property "Value" "GND" (at 95.25 93.98 0)
+      (effects (font (size 1.27 1.27)))
+    )
+    (property "Footprint" "" (at 95.25 88.9 0)
+      (effects (font (size 1.27 1.27)) hide)
+    )
+    (property "Datasheet" "" (at 95.25 88.9 0)
+      (effects (font (size 1.27 1.27)) hide)
+    )
+    (pin "1")
+    (instances
+      (project "voltage_regulated_led_new"
+        (path "/7d837360-0bad-4c76-8645-e18e924dfa75/fdc9af70-ef5e-43c1-851d-2201b5fa75d7"
+          (reference "#PWR011") (unit 1)
+        )
+      )
