File: NEW NEW/voltage_regulated_led_new.kicad_pcb (KiCad board)
At the start: 2 copper layers, 58.4 x 58.4 mm, 11 parts, among them J2 Conn_01x06_Pin, SW2 SW_Push, U1 LM7805_TO220

Commit message: real edits this time!
Parts:
- added SW1: SW_SPST, Button_Switch_THT:SW_DIP_SPSTx01_Piano_10.8x4.1mm_W7.62mm_P2.54mm, F.Cu at (134.6, 106.7)
- J2: value Conn_01x06_Pin -> Conn_01x08_Pin; footprint Connector_PinSocket_2.54mm:PinSocket_1x06_P2.54mm_Vertical -> Connector_PinHeader_2.54mm:PinHeader_1x08_P2.54mm_Vertical
- moved J2 12.7 mm to (147.3, 106.7), turned to 0 degrees
- moved C1 2.54 mm to (127.1, 117.1)
Connections:
- J2 pad 3: GND -> +5V
- J2 pad 6: /Push-Button Activated LED/Vled -> GND
- R1 pad 1: Net-(R1-Pad1) -> GND
- SW2 pad 1: Net-(R1-Pad1) -> GND
Routing:
- net +5V: track 40.4 -> 60.3 mm
- net Net-(R1-Pad1): track 15.9 -> 0.00 mm
- net GND: track 88.4 -> 100.7 mm
- net /+9v: track 0.00 -> 7.62 mm
- net /Push-Button Activated LED/Vled: track 18.0 -> 25.0 mm
- net Net-(D1-K): track 57.9 -> 60.5 mm
- added copper zone on B.Cu, net (none)
