File: NEW NEW/voltage_regulated_led_new.kicad_sch (KiCad schematic)
At the start: 13 parts, among them J1 Conn_01x02_Socket, J2 Conn_01x06_Pin, J4 Conn_01x02_Socket, SW1 SW_SPST, U1 LM7805_TO220

Commit message: real edits this time!
Parts:
- removed J2: Conn_01x06_Pin, Connector_PinSocket_2.54mm:PinSocket_1x06_P2.54mm_Vertical, symbol Connector:Conn_01x06_Pin
- added J2: Conn_01x08_Pin, Connector_PinHeader_2.54mm:PinHeader_1x08_P2.54mm_Vertical, symbol Connector:Conn_01x08_Pin
Connections:
- net +5V: now also J2.3 (Pin_3)
- net +9v: now also J2.1 (Pin_1), J2.2 (Pin_2)
- net GND: now also J2.4 (Pin_4), J2.5 (Pin_5), J2.6 (Pin_6), J2.7 (Pin_7)
- net Push-Button Activated LED/Vled: now also J2.8 (Pin_8)
